File: Senior Design Power PCB.sch (KiCad schematic (older format))
At the start: 10 parts, among them U1 INA226, U2 LM2596S-5

Commit message: Fixed some bugs, added screenshots
Parts:
- C1: value 680uF 50v (N-PL) -> 680uF 35v (Panasonic FK)
- C2: value 330uF 35v (N-PL) -> 680uF 35v (Panasonic FK)
- C3: value 0.01 uF -> 0.1 uF
- D1: value SB540A -> 50WQ04FN
- U2: value LM2596S-5 -> LM2596SX-5
- renumbered R_Sense to RSense
Connections:
- wire segments 71 -> 72
Other:
- moved on the sheet: D1
Changed lines of the file:
@@
 U 1 1 5D7A9EC1
 P 3750 3700
-F 0 "U1" H 3750 4381 50  0000 C CNN
-F 1 "INA226" H 3750 4290 50  0000 C CNN
+F 0 "U1" H 3750 4450 50  0000 C CNN
+F 1 "INA226" H 3750 4350 50  0000 C CNN
 F 2 "Package_SO:VSSOP-10_3x3mm_P0.5mm" H 4550 3250 50  0001 C CNN
 F 3 "http://www.ti.com/lit/ds/symlink/ina226.pdf" H 4100 3600 50  0001 C CNN
@@
 U 1 1 5D7AA788
 P 6250 3500
-F 0 "U2" H 6250 3867 50  0000 C CNN
-F 1 "LM2596S-5" H 6250 3776 50  0000 C CNN
+F 0 "U2" H 5950 3850 50  0000 C CNN
+F 1 "LM2596SX-5" H 6350 3850 50  0000 C CNN
 F 2 "Package_TO_SOT_SMD:TO-263-5_TabPin3" H 6300 3250 50  0001 L CIN
 F 3 "http://www.ti.com/lit/ds/symlink/lm2596.pdf" H 6250 3500 50  0001 C CNN
@@
 U 1 1 5D7AF5DA
 P 7200 3600
-F 0 "L1" H 7200 3815 50  0000 C CNN
-F 1 "33 uH" H 7200 3724 50  0000 C CNN
+F 0 "L1" H 7200 3700 50  0000 C CNN
+F 1 "33 uH" H 7200 3550 50  0000 C CNN
 F 2 "" H 7200 3600 50  0001 C CNN
 F 3 "~" H 7200 3600 50  0001 C CNN
@@
 L Diode:1N5822 D1
 U 1 1 5D7AFE6C
-P 6800 3900
-F 0 "D1" V 6754 3979 50  0000 L CNN
-F 1 "SB540A" V 6845 3979 50  0000 L CNN
-F 2 "Diode_THT:D_DO-201AD_P15.24mm_Horizontal" H 6800 3725 50  0001 C CNN
-F 3 "http://www.vishay.com/docs/88526/1n5820.pdf" H 6800 3900 50  0001 C CNN
-	1    6800 3900
+P 6800 3800
+F 0 "D1" V 6754 3879 50  0000 L CNN
+F 1 "50WQ04FN" V 6845 3879 50  0000 L CNN
+F 2 "Diode_THT:D_DO-201AD_P15.24mm_Horizontal" H 6800 3625 50  0001 C CNN
+F 3 "http://www.vishay.com/docs/88526/1n5820.pdf" H 6800 3800 50  0001 C CNN
+	1    6800 3800
 	0    1    1    0
 $EndComp
@@
 Wire Wire Line
 	7450 3600 7550 3600
-Wire Wire Line
-	7550 3400 6750 3400
 Wire Wire Line
 	6800 4050 6250 4050
@@
 	6800 3600 6950 3600
 Wire Wire Line
-	6800 3600 6800 3750
-Connection ~ 6800 3750
+	6800 3600 6800 3650
 Wire Wire Line
 	6800 3750 6800 3800
 Wire Wire Line
 	6250 3800 6250 4050
-$Comp
-L Device:CP1 C1
-U 1 1 5D7B7A85
-P 5350 3850
-F 0 "C1" H 5465 3896 50  0000 L CNN
-F 1 "680uF 50v (N-PL)" H 5465 3805 50  0000 L CNN
-F 2 "" H 5350 3850 50  0001 C CNN
-F 3 "~" H 5350 3850 50  0001 C CNN
-	1    5350 3850
-	1    0    0    -1
-$EndComp
 $Comp
 L Device:CP1 C2
 U 1 1 5D7B82A7
 P 7550 3850
-F 0 "C2" H 7665 3896 50  0000 L CNN
-F 1 "330uF 35v (N-PL)" H 7665 3805 50  0000 L CNN
+F 0 "C2" H 7500 3600 50  0000 L CNN
+F 1 "680uF 35v (Panasonic FK)" H 7050 3500 50  0000 L CNN
 F 2 "" H 7550 3850 50  0001 C CNN
 F 3 "~" H 7550 3850 50  0001 C CNN
@@
 	3750 3200 3750 3250
 Connection ~ 7550 3400
-Wire Wire Line
-	7550 3400 7550 3500
-$Comp
-L Device:R_US R_Sense
+$Comp
+L Device:R_US RSense
 U 1 1 5D7C461B
 P 2900 3700
-F 0 "R_Sense" H 2968 3746 50  0000 L CNN
-F 1 "0.002 Ohm" H 2968 3655 50  0000 L CNN
+F 0 "RSense" H 2800 3450 50  0000 L CNN
+F 1 "0.002 Ohm" H 2750 3350 50  0000 L CNN
 F 2 "" V 2940 3690 50  0001 C CNN
 F 3 "~" H 2900 3700 50  0001 C CNN
@@
 	3250 3900 3250 4350
 Connection ~ 5350 3400
-Text GLabel 9050 3500 2    50   Input ~ 0
+Text GLabel 8150 3400 2    50   Input ~ 0
 5V
 Wire Wire Line
-	9050 3500 7550 3500
-Connection ~ 7550 3500
-Wire Wire Line
-	7550 3500 7550 3600
-Text GLabel 9050 3700 2    50   Input ~ 0
+	8150 3400 7550 3400
+Text GLabel 8150 3700 2    50   Input ~ 0
 GND
-Text GLabel 9050 3200 2    50   Input ~ 0
+Text GLabel 8150 3100 2    50   Input ~ 0
 SDA
-Text GLabel 9050 3350 2    50   Input ~ 0
+Text GLabel 8150 3250 2    50   Input ~ 0
 SCL
 $Comp
 L power:GND #PWR0103
 U 1 1 5D7D0F22
-P 9000 3950
-F 0 "#PWR0103" H 9000 3700 50  0001 C CNN
-F 1 "GND" H 9005 3777 50  0000 C CNN
-F 2 "" H 9000 3950 50  0001 C CNN
-F 3 "" H 9000 3950 50  0001 C CNN
-	1    9000 3950
-	1    0    0    -1
-$EndComp
-Wire Wire Line
-	9050 3700 9000 3700
-Wire Wire Line
-	9000 3700 9000 3950
+P 8100 3950
+F 0 "#PWR0103" H 8100 3700 50  0001 C CNN
+F 1 "GND" H 8105 3777 50  0000 C CNN
+F 2 "" H 8100 3950 50  0001 C CNN
+F 3 "" H 8100 3950 50  0001 C CNN
+	1    8100 3950
+	1    0    0    -1
+$EndComp
+Wire Wire Line
+	8150 3700 8100 3700
+Wire Wire Line
+	8100 3700 8100 3950
 $Comp
 L Device:R_US R1
@@
 Wire Wire Line
 	4350 3300 4350 3100
-Wire Wire Line
-	3750 3100 4350 3100
 Connection ~ 4350 3100
 Wire Wire Line
@@
 Wire Wire Line
 	5050 4350 5050 3400
-Wire Wire Line
-	3250 4350 4550 4350
 Wire Wire Line
 	5050 3400 5350 3400
@@
 Wire Wire Line
 	4950 3700 4950 3200
-Wire Wire Line
-	4950 3200 9050 3200
 Connection ~ 4350 3700
 Wire Wire Line
-	8700 3350 8700 3300
-Wire Wire Line
-	8700 3300 4850 3300
-Wire Wire Line
-	4850 3300 4850 3800
-Wire Wire Line
 	4850 3800 4700 3800
-Wire Wire Line
-	8700 3350 9050 3350
 Connection ~ 4700 3800
 Text GLabel 2500 3450 0    50   Input ~ 0
@@
 P 4550 4050
 F 0 "C3" H 4665 4096 50  0000 L CNN
-F 1 "0.01 uF" H 4665 4005 50  0000 L CNN
+F 1 "0.1 uF" H 4665 4005 50  0000 L CNN
 F 2 "" H 4588 3900 50  0001 C CNN
 F 3 "~" H 4550 4050 50  0001 C CNN
@@
 $EndComp
 Wire Wire Line
-	4550 4350 4550 4200
-Connection ~ 4550 4350
-Wire Wire Line
-	4550 4350 5050 4350
-Wire Wire Line
 	4550 3900 4550 3100
 Connection ~ 4550 3100
 Wire Wire Line
 	4550 3100 4700 3100
+$Comp
+L Device:CP1 C1
+U 1 1 5D7B7A85
+P 5350 3850
+F 0 "C1" H 5300 3600 50  0000 L CNN
+F 1 "680uF 35v (Panasonic FK)" H 5100 3500 50  0000 L CNN
+F 2 "" H 5350 3850 50  0001 C CNN
+F 3 "~" H 5350 3850 50  0001 C CNN
+	1    5350 3850
+	1    0    0    -1
+$EndComp
+Wire Wire Line
+	6800 4050 6800 3950
+Wire Wire Line
+	4850 3250 4850 3800
+Wire Wire Line
+	6750 3400 7550 3400
+Wire Wire Line
+	7550 3400 7550 3600
+Wire Wire Line
+	4250 3100 4350 3100
+Wire Wire Line
+	3750 3100 4350 3100
+Wire Wire Line
+	8150 3250 4850 3250
+Wire Wire Line
+	8150 3100 7950 3100
+Wire Wire Line
+	7950 3100 7950 3200
+Wire Wire Line
+	7950 3200 4950 3200
+Wire Wire Line
+	3250 4350 5050 4350
+Wire Wire Line
+	4550 4200 4550 4250
+Wire Wire Line
+	4550 4250 4200 4250
+Connection ~ 4200 4250
 $EndSCHEMATC
