File: Senior Design Power PCB.kicad_pcb (KiCad board)
At the start: 2 copper layers, 70.1 x 32 mm, 16 parts, among them U2 TO-263-5_TabPin3, U2 VSSOP-10_3x3mm_P0.5mm

Commit message: Fixed some bugs, added screenshots
Parts:
- renumbered U2 to U1
Connections:
- C1 pad 2: (no net) -> B-
Routing:
- net 5V: track 106.7 -> 103.9 mm
Changed lines of the file:
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@@
-(kicad_pcb (version 20171130) (host pcbnew 5.1.4-e60b266~84~ubuntu18.04.1)
+(kicad_pcb (version 20171130) (host pcbnew "(5.1.4)-1")
   (general
     (thickness 1.6)
     (drawings 15)
-    (tracks 156)
+    (tracks 155)
     (zones 0)
     (modules 16)
@@
     (solder_mask_min_width 0.25)
     (aux_axis_origin 0 0)
-    (visible_elements FFFFFF7F)
+    (visible_elements 7FFFFFFF)
     (pcbplotparams
       (layerselection 0x010fc_ffffffff)
@@
     (fp_circle (center 2.5 0) (end 7.62 0) (layer F.SilkS) (width 0.12))
     (fp_circle (center 2.5 0) (end 7.5 0) (layer F.Fab) (width 0.1))
-    (pad 2 thru_hole circle (at 5 0 270) (size 2 2) (drill 1) (layers *.Cu *.Mask))
+    (pad 2 thru_hole circle (at 5 0 270) (size 2 2) (drill 1) (layers *.Cu *.Mask)
+      (net 1 B-))
     (pad 1 thru_hole rect (at 0 0 270) (size 2 2) (drill 1) (layers *.Cu *.Mask)
       (net 5 B+))
@@
     (tags "resistor handsolder")
     (attr smd)
-    (fp_text reference R2 (at 3.302 -1.016) (layer F.SilkS)
+    (fp_text reference R2 (at 3.302 0.254) (layer F.SilkS)
       (effects (font (size 1 1) (thickness 0.15)))
     )
@@
     (tags "VSSOP SO")
     (attr smd)
-    (fp_text reference U2 (at 0 -2.45) (layer F.SilkS)
+    (fp_text reference U1 (at 0 -2.45) (layer F.SilkS)
       (effects (font (size 1 1) (thickness 0.15)))
     )
@@
   (segment (start 27.568 44.285) (end 27.568 42.037) (width 0.2) (layer F.Cu) (net 4))
   (segment (start 27.568 44.196) (end 27.568 43.396) (width 0.2) (layer F.Cu) (net 4))
-  (segment (start 27.568 44.196) (end 28.243 44.196) (width 0.2) (layer F.Cu) (net 4))
   (segment (start 31.75 40.268) (end 31.75 45.085) (width 0.2) (layer F.Cu) (net 4))
   (segment (start 27.568 42.037) (end 27.568 38.998) (width 0.2) (layer F.Cu) (net 4))
   (segment (start 31.623 45.085) (end 31.75 45.085) (width 0.2) (layer F.Cu) (net 4))
-  (segment (start 28.243 45.085) (end 31.623 45.085) (width 0.2) (layer F.Cu) (net 4))
   (segment (start 73.867 40.974) (end 82.296 40.974) (width 3) (layer F.Cu) (net 4))
   (segment (start 70.358 37.465) (end 73.867 40.974) (width 3) (layer F.Cu) (net 4))
@@
   (segment (start 39.878 43.688) (end 34.036 43.688) (width 0.25) (layer B.Cu) (net 4))
   (segment (start 43.942 39.624) (end 39.878 43.688) (width 0.25) (layer B.Cu) (net 4))
+  (segment (start 64.77 26.69) (end 64.77 27.94) (width 0.25) (layer F.Cu) (net 4))
   (segment (start 27.6 37.846) (end 27.6 37.346) (width 0.2) (layer F.Cu) (net 5))
   (segment (start 39.5875 25.146) (end 39.5875 28.7385) (width 0.25) (layer F.Cu) (net 5))
